Commit message: update

File: jaco_model/urdf/mico_arm.xacro (robot description, xacro)
@@ -105,28 +105,194 @@
     <property name="end_effector_offset" value="0.160"/>
     <property name="link_base_link_data">
-        <xacro:default_link_data link_name="${link_base}"/>
+        <!--<xacro:default_link_data link_name="${link_base}"/>-->
+        <link_data>
+            <collision>
+                <geometry>
+                    <mesh filename="package://jaco_model/meshes/${link_base}.dae"/>
+                </geometry>
+            </collision>
+            <inertial>
+                <origin xyz="0 0 0" rpy="0 0 0"/>
+                <mass value="1.409835"/>
+                <inertia ixx="0.299757" ixy="0.0" ixz="0.0"
+                         iyy="0.299811" iyz="0.0"
+                         izz="0.124476"/>
+            </inertial>
+        </link_data>
     </property>
     <property name="link_1_link_data">
-        <xacro:default_link_data link_name="${link_1}"/>
+        <!--<xacro:default_link_data link_name="${link_1}"/>-->
+        <link_data>
+            <collision>
+                <geometry>
+                    <mesh filename="package://jaco_model/meshes/${link_1}.dae"/>
+                </geometry>
+            </collision>
+            <inertial>
+                <origin xyz="0 0 0" rpy="0 0 0"/>
+                <mass value="1.08"/>
+                <inertia ixx="0.265738" ixy="0.0" ixz="0.0"
+                         iyy="0.273832" iyz="0.036701"
+                         izz="0.076209"/>
+            </inertial>
+        </link_data>
     </property>
     <property name="link_2_link_data">
-        <xacro:default_link_data link_name="${link_2}"/>
+        <!--<xacro:default_link_data link_name="${link_2}"/>-->
+        <link_data>
+            <collision>
+                <geometry>
+                    <mesh filename="package://jaco_model/meshes/${link_2}.dae"/>
+                </geometry>
+            </collision>
+            <inertial>
+                <origin xyz="0 0 0" rpy="0 0 0"/>
+                <mass value="1.642299"/>
+                <inertia ixx="0.080532" ixy="0.0" ixz="0.0"
+                         iyy="2.112210" iyz="0.0"
+                         izz="2.155361"/>
+            </inertial>
+        </link_data>
     </property>
     <property name="link_3_link_data">
-        <xacro:default_link_data link_name="${link_3}"/>
+        <!--<xacro:default_link_data link_name="${link_3}"/>-->
+        <link_data>
+            <collision>
+                <geometry>
+                    <mesh filename="package://jaco_model/meshes/${link_3}.dae"/>
+                </geometry>
+            </collision>
+            <inertial>
+                <origin xyz="0 0 0" rpy="0 0 0"/>
+                <mass value="0.815865"/>
+                <inertia ixx="0.042395" ixy="0.0" ixz="-0.015301"
+                         iyy="0.207338" iyz="0.0"
+                         izz="0.219274"/>
+            </inertial>
+        </link_data>
     </property>
     <property name="link_4_link_data">
-        <xacro:default_link_data link_name="${link_4}"/>
+        <!--<xacro:default_link_data link_name="${link_4}"/>-->
+        <link_data>
+            <collision>
+                <geometry>
+                    <mesh filename="package://jaco_model/meshes/${link_4}.dae"/>
+                </geometry>
+            </collision>
+            <inertial>
+                <origin xyz="0 0 0" rpy="0 0 0"/>
+                <mass value="0.450840"/>
+                <inertia ixx="0.032664" ixy="0.0" ixz="0.007368"
+                         iyy="0.035487" iyz="0.0"
+                         izz="0.024157"/>
+            </inertial>
+        </link_data>
     </property>
     <property name="link_5_link_data">
-        <xacro:default_link_data link_name="${link_5}"/>
+        <!--<xacro:default_link_data link_name="${link_5}"/>-->
+        <link_data>
+            <collision>
+                <geometry>
+                    <mesh filename="package://jaco_model/meshes/${link_5}.dae"/>
+                </geometry>
+            </collision>
+            <inertial>
+                <origin xyz="0 0 0" rpy="0 0 0"/>
+                <mass value="0.450840"/>
+                <inertia ixx="0.032664" ixy="0.0" ixz="0.007368"
+                         iyy="0.035487" iyz="0.0"
+                         izz="0.024157"/>
+            </inertial>
+        </link_data>
     </property>
     <property name="link_hand_link_data">
-        <xacro:default_link_data link_name="${link_hand}"/>
+        <!--<xacro:default_link_data link_name="${link_hand}"/>-->
+        <link_data>
+            <collision>
+                <geometry>
+                    <mesh filename="package://jaco_model/meshes/${link_hand}.dae"/>
+                </geometry>
+            </collision>
+            <inertial>
+                <origin xyz="0 0 0" rpy="0 0 0"/>
+                <mass value="1.0e-2"/>
+                <inertia ixx="1.0e-5" ixy="0.0" ixz="0.0"
+                         iyy="1.0e-5" iyz="0.0"
+                         izz="1.0e-5"/>
+            </inertial>
+        </link_data>
+    </property>
+    <property name="link_finger_1_link_data">
+        <!--<xacro:default_link_data link_name="${link_hand}"/>-->
+        <link_data>
+            <collision>
+                <geometry>
+                    <mesh filename="package://jaco_model/meshes/${link_finger_1}.dae"/>
+                </geometry>
+            </collision>
+            <inertial>
+                <origin xyz="0 0 0" rpy="0 0 0"/>
+                <mass value="1.0e-2"/>
+                <inertia ixx="1.0e-5" ixy="0.0" ixz="0.0"
+                         iyy="1.0e-5" iyz="0.0"
+                         izz="1.0e-5"/>
+            </inertial>
+        </link_data>
+    </property>
+    <property name="link_finger_tip_1_link_data">
+        <!--<xacro:default_link_data link_name="${link_hand}"/>-->
+        <link_data>
+            <collision>
+                <geometry>
+                    <mesh filename="package://jaco_model/meshes/${link_finger_tip_1}.dae"/>
+                </geometry>
+            </collision>
+            <inertial>
+                <origin xyz="0 0 0" rpy="0 0 0"/>
+                <mass value="1.0e-2"/>
+                <inertia ixx="1.0e-5" ixy="0.0" ixz="0.0"
+                         iyy="1.0e-5" iyz="0.0"
+                         izz="1.0e-5"/>
+            </inertial>
+        </link_data>
+    </property>
+    <property name="link_finger_2_link_data">
+        <!--<xacro:default_link_data link_name="${link_hand}"/>-->
+        <link_data>
+            <collision>
+                <geometry>
+                    <mesh filename="package://jaco_model/meshes/${link_finger_2}.dae"/>
+                </geometry>
+            </collision>
+            <inertial>
+                <origin xyz="0 0 0" rpy="0 0 0"/>
+                <mass value="1.0e-2"/>
+                <inertia ixx="1.0e-5" ixy="0.0" ixz="0.0"
+                         iyy="1.0e-5" iyz="0.0"
+                         izz="1.0e-5"/>
+            </inertial>
+        </link_data>
+    </property>
+    <property name="link_finger_tip_2_link_data">
+        <!--<xacro:default_link_data link_name="${link_hand}"/>-->
+        <link_data>
+            <collision>
+                <geometry>
+                    <mesh filename="package://jaco_model/meshes/${link_finger_tip_2}.dae"/>
+                </geometry>
+            </collision>
+            <inertial>
+                <origin xyz="0 0 0" rpy="0 0 0"/>
+                <mass value="1.0e-2"/>
+                <inertia ixx="1.0e-5" ixy="0.0" ixz="0.0"
+                         iyy="1.0e-5" iyz="0.0"
+                         izz="1.0e-5"/>
+            </inertial>
+        </link_data>
     </property>
     <xacro:macro name="mico_arm" params="parent">
         <xacro:jaco_struct parent="${parent}" basename="mico"/>
         <xacro:jaco_link link_name="${link_finger_1}">
-            <xacro:default_link_data link_name="${link_finger_1}"/>
+            <xacro:insert_block name="link_finger_1_link_data"/>
         </xacro:jaco_link>
         <xacro:jaco_finger_joint joint_name="${joint_finger_1}" type="revolute" parent="${link_hand}"
@@ -137,5 +303,5 @@
                                  upper_limit="${joint_finger_1_upper_limit}"/>
         <xacro:jaco_link link_name="${link_finger_tip_1}">
-            <xacro:default_link_data link_name="${link_finger_tip_1}"/>
+            <xacro:insert_block name="link_finger_tip_1_link_data"/>
         </xacro:jaco_link>
         <xacro:jaco_finger_tip_joint joint_name="${joint_finger_tip_1}" type="revolute" parent="${link_finger_1}"
@@ -148,5 +314,5 @@
                                      mimic_offset="${joint_finger_tip_1_mimc_offset}"/>
         <xacro:jaco_link link_name="${link_finger_2}">
-            <xacro:default_link_data link_name="${link_finger_2}"/>
+            <xacro:insert_block name="link_finger_2_link_data"/>
         </xacro:jaco_link>
         <xacro:jaco_finger_joint joint_name="${joint_finger_2}" type="revolute" parent="${link_hand}"
@@ -157,5 +323,5 @@
                                  upper_limit="${joint_finger_2_upper_limit}"/>
         <xacro:jaco_link link_name="${link_finger_tip_2}">
-            <xacro:default_link_data link_name="${link_finger_tip_2}"/>
+            <xacro:insert_block name="link_finger_tip_2_link_data"/>
         </xacro:jaco_link>
         <xacro:jaco_finger_tip_joint joint_name="${joint_finger_tip_2}" type="revolute" parent="${link_finger_2}"
